File: fresh_air_controller/electrical/fresh_air_controller/_autosave-fresh_air_controller_board.sch (KiCad schematic (older format))
At the start: 28 parts

Commit message: use analog_threshold for monitor and garage doors. update some pinout for fresh air controller.
Parts:
- removed U? (x5): PCF8574_RelayMod, symbol birkler_comp:PCF8574_RelayMod
- added C?: CP, symbol Device:CP
- added K? (x5): FINDER-34.51, Relay_THT:Relay_SPDT_Finder_34.51_Vertical, symbol Relay:FINDER-34.51
- added R? (x5): 10K, symbol Device:R
Connections:
- net labels removed: NC0, NC1
- wire segments 170 -> 204
Other:
- moved on the sheet: J?, R?, U?
